File: 6802Slave/6802-2slv.sch (KiCad schematic (older format))
At the start: 68 parts, among them J1 DB15, J2 USB B conn., J3 USB A connector, J4 ICSP, P1 CONN_1, U1 LTC6802-2, U2 TCLT1009, U3 ACPL-W61L, U4 ACPL-K64L, U5 PIC16F1825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

Commit message: fixed schematic comments
Other:
- note added: "For temperature sensor 1 on J1-pin15, \nomit R29 when using diodes. If using \nthermistor, add R29 to circuit.\n\nFor temperature sensor 2 on J1-pin8, \nomit R30 when using diodes. If using \nthermistor, add R30 to circuit."
- note removed: "For temperature sensor 1 on J1-pin15, \nomit R29 when using diodes. If using \nthermistor, add R14a to circuit.\n\nFor temperature sensor 2 on J1-pin8, \nomit R30 when using diodes. If using \nthermistor, add R15a to circuit."
Changed lines of the file:
@@
-EESchema Schematic File Version 2  date 18/03/2013 14:37:45
+EESchema Schematic File Version 2  date 23/03/2013 20:33:18
 LIBS:power
 LIBS:device
@@
 Sheet 1 1
 Title "LTC6802-2 based slave cell monitor"
-Date "17 mar 2013"
+Date "23 mar 2013"
 Rev "D"
 Comp "www.go-ev.co.uk"
@@
 	5400 5550 5400 4700
 Text Notes 5400 5700 0    60   ~ 0
-For temperature sensor 1 on J1-pin15, \nomit R29 when using diodes. If using \nthermistor, add R14a to circuit.\n\nFor temperature sensor 2 on J1-pin8, \nomit R30 when using diodes. If using \nthermistor, add R15a to circuit.
+For temperature sensor 1 on J1-pin15, \nomit R29 when using diodes. If using \nthermistor, add R29 to circuit.\n\nFor temperature sensor 2 on J1-pin8, \nomit R30 when using diodes. If using \nthermistor, add R30 to circuit.
 $Comp
 L R R27
