File: 6802Slave/6802-2slv.kicad_pcb (KiCad board)
At the start: 2 copper layers, 68 parts, among them J1 DB15, J2 USB B conn., J3 USB A connector, J4 ICSP, P1 CONN_1, U1 LTC6802-2, U2 TCLT1009, U3 ACPL-W61L, U4 ACPL-K64L, U5 PIC16F1825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

Commit message: layout work
Parts:
- moved U2 37.8 mm to (208.2, 194.5), turned to 270 degrees
- moved R29 36.5 mm to (237.0, 212.0)
- moved R30 36.0 mm to (240.5, 212.0)
- moved C16 25.3 mm to (206.5, 203.5), turned to 270 degrees
- moved R18 20.5 mm to (210.0, 202.2), turned to 90 degrees
- moved D1 18.8 mm to (264.5, 154.5)
- moved J2 18.8 mm to (277.0, 159.0)
- moved J3 18.8 mm to (251.0, 161.0)
- moved J4 18.8 mm to (224.0, 154.5)
- moved R24 18.8 mm to (239.0, 164.5)
- moved R27 18.8 mm to (246.0, 164.5)
- moved R28 18.8 mm to (248.0, 164.5)
- moved R16 17.5 mm to (203.8, 204.0), turned to 270 degrees
- moved R17 13.6 mm to (226.8, 203.0), turned to 270 degrees
- moved U3 12.1 mm to (230.0, 193.8), turned to 0 degrees
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Routing:
- net N-0000065: track 0.00 -> 21.6 mm
- net N-0000014: track 0.00 -> 20.6 mm
- net GNDPWR: track 0.00 -> 18.3 mm, vias 0 -> 13
- net N-0000083: track 0.00 -> 17.1 mm
- net N-0000066: track 0.00 -> 15.5 mm
- net N-0000011: track 0.00 -> 15.5 mm
- net N-0000012: track 0.00 -> 14.6 mm
- net N-0000016: track 0.00 -> 13.0 mm
- net N-0000013: track 0.00 -> 12.4 mm
- net N-0000017: track 0.00 -> 11.6 mm
- net N-0000081: track 0.00 -> 11.5 mm
- net N-0000010: track 0.00 -> 10.6 mm
- net N-0000020: track 0.00 -> 10.5 mm
- net N-0000033: track 0.00 -> 10.2 mm
- net N-0000022: track 0.00 -> 10.2 mm
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Other:
- rule trace_min: 0.254 -> 0.2

Commit message: more pcb layout
Parts:
- moved P1 34.5 mm to (232.8, 202.5)
- moved R18 19.3 mm to (229.2, 203.5), turned to 270 degrees
- moved C18 6.25 mm to (237.0, 203.5), turned to 90 degrees
- moved C17 5.00 mm to (239.2, 203.5), turned to 90 degrees
- moved R29 3.75 mm to (240.8, 212.0)
- moved R30 3.50 mm to (237.0, 212.0), turned to 90 degrees
- moved R16 1.58 mm to (204.2, 202.5)
- moved R17 0.71 mm to (227.2, 203.5)
- moved C16 0.50 mm to (206.5, 203.0), turned to 90 degrees
- moved U2 0.25 mm to (208.0, 194.5)
Routing:
- net N-0000087: track 0.00 -> 61.0 mm
- net N-0000053: track 0.00 -> 52.2 mm
- net N-0000083: track 17.1 -> 54.0 mm
- net N-0000066: track 15.5 -> 49.2 mm, vias 0 -> 1
- net N-0000056: track 0.00 -> 30.3 mm
- net N-0000065: track 21.6 -> 49.3 mm
- net N-0000057: track 0.00 -> 27.5 mm
- net GNDPWR: track 18.3 -> 36.7 mm, vias 13 -> 17
- net N-000002: track 2.68 -> 19.8 mm
- net N-000001: track 0.00 -> 10.6 mm
- net N-0000054: track 0.00 -> 4.71 mm
- net N-0000055: track 0.00 -> 4.62 mm

Commit message: pcb layout nearly finished
Parts:
- moved C22 148.3 mm to (147.3, 134.3), turned to 90 degrees
- moved J2 147.8 mm to (139.4, 105.0), turned to 270 degrees
- moved R26 147.1 mm to (139.6, 115.3), turned to 0 degrees
- moved C25 146.6 mm to (147.3, 130.1)
- moved R25 143.9 mm to (139.6, 118.3), turned to 0 degrees
- moved C20 143.7 mm to (151.6, 108.3)
- moved D2 141.3 mm to (147.3, 125.6), turned to 90 degrees
- moved C23 140.5 mm to (150.8, 122.6)
- moved C21 140.1 mm to (151.6, 135.1)
- moved C24 138.6 mm to (155.8, 135.1), turned to 180 degrees
- moved R22 138.0 mm to (158.3, 100.8), turned to 0 degrees
- moved R23 138.0 mm to (158.3, 102.8), turned to 180 degrees
- moved U6 136.5 mm to (155.1, 129.3), turned to 0 degrees
- moved U5 135.7 mm to (151.6, 114.6), turned to 270 degrees
- moved D1 134.2 mm to (135.8, 116.4), turned to 90 degrees
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Routing:
- net N-0000085: track 0.00 -> 113.8 mm
- net N-0000046: track 0.00 -> 73.1 mm
- net N-0000027: track 0.00 -> 41.4 mm
- net GND: track 0.00 -> 37.2 mm, vias 0 -> 5
- net N-0000052: track 0.00 -> 31.0 mm, vias 0 -> 1
- net N-0000043: track 0.00 -> 20.1 mm, vias 0 -> 2
- net N-0000058: track 0.00 -> 18.7 mm
- net N-0000041: track 0.00 -> 18.1 mm, vias 0 -> 2
- net N-0000064: track 0.00 -> 16.3 mm
- net N-0000042: track 0.00 -> 16.1 mm, vias 0 -> 2
- net N-0000062: track 0.00 -> 15.9 mm
- net N-0000044: track 0.00 -> 15.3 mm
- net N-0000051: track 0.00 -> 14.4 mm
- net N-0000035: track 0.00 -> 13.9 mm
- net N-0000045: track 0.00 -> 13.6 mm, vias 0 -> 2
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- added copper zone on B.Cu, net GND
- added copper zone on B.Cu, net GNDPWR
- added copper zone on B.Cu, net N-0000088
Other:
- board text added: "DANGER! HIGH VOLTAGE!"
- board text added: "Licensed under the TAPR Open Hardware License (www.tapr.org/OHL)"
- board text added: "Temp 2 Temp 1 Cell 1- Cell 1+ Cell 2+ Cell 3+ Cell 4+ Cell 5+ Cell 6+ Cell 7+ Cell 8+ Cell 9+ Cell 10+ Cell 11+ Cell 12+"
- board text added: "evBMS LTC6802-2 cell monitor (c) Greg Fordyce 2013 - Rev D"
