File: 6802Slave/6802-2slv.kicad_pcb (KiCad board)
At the start: 2 copper layers, 68 parts, among them J1 DB15, J2 USB B conn., J3 USB A connector, J4 ICSP, P1 CONN_1, U1 LTC6802-2, U2 TCLT1009, U3 ACPL-W61L, U4 ACPL-K64L, U5 PIC16F1825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

Commit message: More pcb updates
Other:
- board text added: "DANGER!"
- board text added: "HIGH VOLTAGE!"
Changed lines of the file:
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@@
     (links 152)
     (no_connects 0)
-    (area 124.64557 90.299999 213.396401 145.300001)
+    (area 124.64557 90.299999 213.396401 144.200001)
     (thickness 1.6)
-    (drawings 89)
+    (drawings 84)
     (tracks 703)
     (zones 0)
@@
     (descr "Connecteur DB15 MALE couche")
     (tags "CONN DB15")
-    (fp_text reference J1 (at 21.5 -1 270) (layer F.SilkS)
+    (fp_text reference J1 (at 16.775 -4.525 270) (layer F.SilkS)
       (effects (font (size 1.524 1.524) (thickness 0.3048)))
     )
@@
     )
   )
+  (gr_text DANGER! (at 187.7 95.5) (layer F.SilkS)
+    (effects (font (size 2 2) (thickness 0.35)))
+  )
+  (gr_text "HIGH VOLTAGE!" (at 187.2 140.3) (layer F.SilkS)
+    (effects (font (size 2 2) (thickness 0.35)))
+  )
+  (gr_line (start 167 142) (end 167 94) (angle 90) (layer F.SilkS) (width 0.2))
+  (gr_line (start 174.1 142.8) (end 200.9 142.8) (angle 90) (layer Eco2.User) (width 0.2))
+  (gr_line (start 174.1 92.8) (end 200.9 92.8) (angle 90) (layer Eco2.User) (width 0.2))
   (gr_line (start 204.1 142.8) (end 206 142.8) (angle 90) (layer Eco2.User) (width 0.2))
-  (gr_line (start 181.9 142.8) (end 200.9 142.8) (angle 90) (layer Eco2.User) (width 0.2))
-  (gr_line (start 175.9 142.8) (end 175.9 142.7) (angle 90) (layer Eco2.User) (width 0.2))
-  (gr_line (start 174.1 142.8) (end 175.9 142.8) (angle 90) (layer Eco2.User) (width 0.2))
   (gr_line (start 134.1 142.8) (end 170.9 142.8) (angle 90) (layer Eco2.User) (width 0.2))
   (gr_line (start 130.9 142.8) (end 129 142.8) (angle 90) (layer Eco2.User) (width 0.2))
@@
   (gr_line (start 170.9 94.7) (end 170.9 92.8) (angle 90) (layer Eco2.User) (width 0.2))
   (gr_line (start 174.1 92.8) (end 174.1 94.8) (angle 90) (layer Eco2.User) (width 0.2))
-  (gr_line (start 176 92.8) (end 174.1 92.8) (angle 90) (layer Eco2.User) (width 0.2))
-  (gr_line (start 200.9 92.8) (end 181.9 92.8) (angle 90) (layer Eco2.User) (width 0.2))
   (gr_line (start 200.9 94.7) (end 200.9 92.8) (angle 90) (layer Eco2.User) (width 0.2))
   (gr_line (start 204.1 92.8) (end 206 92.8) (angle 90) (layer Eco2.User) (width 0.2))
@@
   (gr_line (start 206 140.6) (end 206 95.2) (angle 90) (layer Eco2.User) (width 0.2))
   (gr_line (start 129 140.6) (end 129 95.2) (angle 90) (layer Eco2.User) (width 0.2))
-  (gr_line (start 175.6 90.4) (end 175.6 90.5) (angle 90) (layer Eco2.User) (width 0.2))
-  (gr_arc (start 178.9 91.4) (end 182.2 91.4) (angle 90) (layer Eco2.User) (width 0.2))
-  (gr_arc (start 178.9 91.4) (end 178.9 94.7) (angle 90) (layer Eco2.User) (width 0.2))
-  (gr_arc (start 178.9 144.1) (end 175.6 144.1) (angle 90) (layer Eco2.User) (width 0.2))
-  (gr_arc (start 178.9 144.1) (end 178.9 140.8) (angle 90) (layer Eco2.User) (width 0.2))
   (gr_text "     DANGER!  \nHIGH VOLTAGE!" (at 172 115 90) (layer B.SilkS)
     (effects (font (size 3 3) (thickness 0.5)) (justify mirror))
@@
     (effects (font (size 1 1) (thickness 0.15)) (justify mirror))
   )
-  (gr_text "evBMS LTC6802-2 cell monitor \n (c) Greg Fordyce 2013 - Rev D " (at 154.7 140.7) (layer F.SilkS)
+  (gr_text "evBMS LTC6802-2 cell monitor \n (c) Greg Fordyce 2013 - Rev D " (at 152.9 139.3) (layer F.SilkS)
     (effects (font (size 1 1) (thickness 0.15)))
   )
-  (gr_text " Licensed under the \nTAPR Open Hardware License \n (www.tapr.org/OHL)" (at 153.5 92.6) (layer F.SilkS)
+  (gr_text " Licensed under the \nTAPR Open Hardware License \n (www.tapr.org/OHL)" (at 153.7 94.6) (layer F.SilkS)
     (effects (font (size 1 1) (thickness 0.15)))
   )
